File: 2240-breakout.kicad_sch (KiCad schematic)
At the start: 16 parts, among them J1 Conn_01x04_Pin, U1 TMC2240ATJ+

Commit message: did some stuff
Parts:
- added D1: LED, symbol Device:LED
- added J2: Conn_01x05_Pin, symbol Connector:Conn_01x05_Pin
- added Q1, Q2: NMOS, symbol Simulation_SPICE:NMOS
- added R1, R2, R3: 100k, symbol Device:R
- added R4, R5: 10k, symbol Device:R
- added R6: R, symbol Device:R
- added TP5, TP6, TP7, TP8: TestPoint, symbol Connector:TestPoint
Connections:
- net GND: now also J2.5 (Pin_5), Q1.3 (S), Q2.3 (S), R1.2, R2.2, R3.2
- net +3.3V: now reaches C7.1, U1.5 (VCC_IO)
- net +3.3V: now also J2.1 (Pin_1), R4.1, R5.1, R6.1
- net +1V8: now reaches C10.1, U1.3 (VDD1V8)
- net OV#: now reaches U1.13 (OV)
- net OV#: now also Q1.2 (G), R4.2
- net SPI_CS#: now reaches U1.26 (CSN/AD2)
- net SPI_CS#: now also TP8.1
- net SPI_SCK: now reaches U1.27 (SCK/AD1)
- net SPI_SCK: now also TP5.1
- net SPI_SDI: now reaches U1.28 (SDI/AD0)
- net SPI_SDI: now also TP6.1
- net SPI_SDO: now reaches U1.29 (SDO/NAO)
- net SPI_SDO: now also TP7.1
- net ENCN: now reaches U1.6 (ENCN)
- net ENCN: now also J2.4 (Pin_4), R1.1
- net ENCB: now reaches U1.7 (ENCB)
- net ENCB: now also J2.3 (Pin_3), R2.1
- net ENCA: now reaches U1.8 (ENCA)
- net ENCA: now also J2.2 (Pin_2), R3.1
- new net: D1.1 (K), Q2.1 (D)
- new net: D1.2 (A), R6.2
- new net OV_AH: Q1.1 (D), Q2.2 (G), R5.2
Other:
- moved on the sheet: C1, C10, C2, C3, C4, C5, C6, C7, C8, C9, J1, TP1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
