File: tmc2240-breakout.kicad_pcb (KiCad board)
At the start: 2 copper layers, 60 x 60 mm, 91 parts, among them J1 Conn_01x06, J2 Conn_01x05, J3 Conn_01x02, J4 Conn_01x02, J5 Conn_01x17, J6 Conn_01x06, J7 Conn_01x05, J8 Conn_01x02, Q10 2N7002, Q11 2N7002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

Commit message: did some layouting
Routing:
- net (no net): track 2.12 -> 3.43 mm
Changed lines of the file:
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@@
+	)
+	(segment
+		(start 130.75 76.75)
+		(end 130 76)
+		(width 0.2)
+		(layer "F.Cu")
+		(net 0)
 	)
 	(segment
@@
 		(width 0.2)
 		(layer "F.Cu")
+		(net 0)
+	)
+	(segment
+		(start 130 76)
+		(end 130 75.75)
+		(width 0.2)
+		(layer "F.Cu")
