File: tmc2240-breakout.kicad_pcb (KiCad board)
At the start: 2 copper layers, 60 x 60 mm, 91 parts, among them J1 Conn_01x06, J2 Conn_01x05, J3 Conn_01x02, J4 Conn_01x02, J5 Conn_01x17, J6 Conn_01x06, J7 Conn_01x05, J8 Conn_01x02, Q10 2N7002, Q11 2N7002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

Commit message: more layouting
Parts:
- moved C11 7.30 mm to (132.5, 112.2), turned to 90 degrees
- moved C10 0.56 mm to (141.0, 88.2), turned to -90 degrees
- moved C7 0.25 mm to (141.0, 90.8), turned to 90 degrees
Routing:
- net /IREF: track 28.3 -> 97.7 mm, vias 0 -> 1
- net /IREF_R2: track 1.82 -> 46.6 mm
- net /IREF_R3: track 5.72 -> 49.6 mm
- net GND: track 16.2 -> 25.8 mm, vias 14 -> 29
- net Net-(Q3-D): track 0.00 -> 5.48 mm
- net +1V8: track 2.64 -> 0.00 mm
- net +3.3V: track 2.22 -> 0.00 mm, vias 0 -> 4
- net (no net): track 3.43 -> 2.12 mm
- net /ENCA: track 35.4 -> 34.4 mm
- net /ENCB: track 35.3 -> 34.5 mm
- net /DIR: track 26.1 -> 26.8 mm
- net /ENCN: track 36.9 -> 36.2 mm
- net /DRV_EN#: track 29.4 -> 28.7 mm, vias 0 -> 2
- net /UART_EN: track 29.1 -> 28.5 mm, vias 0 -> 2
- net /DIAG0#: vias 0 -> 2
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
Commit message: more pcb layout
Routing:
- net +3.3V: track 0.00 -> 134.1 mm
- net /OV: track 32.7 -> 83.3 mm, vias 2 -> 4
- net /DRV_EN#: track 28.7 -> 53.4 mm, vias 2 -> 4
- net GND: track 25.8 -> 26.9 mm, vias 29 -> 51
- net /SLEEP#: track 50.3 -> 50.2 mm, vias 0 -> 1
- net VMOTOR: vias 5 -> 28

Commit message: did some more layouting
Routing:
- net /DIAG1#: track 30.2 -> 68.1 mm, vias 2 -> 6
- net /DIAG0#: track 28.7 -> 63.4 mm, vias 2 -> 6
- net /DIAG0_AH: track 10.6 -> 11.4 mm
Other:
- board text removed: "TODO: Motor pin labels are wrong"

Commit message: more pcb layouting
Parts:
- moved R1 2.70 mm to (143.8, 100.0)
- moved R3 2.50 mm to (146.5, 100.0)
Connections:
- net Net-(Q9-D) renamed /OV_D
- net Net-(U1A-CLK) renamed /CLK
- J2 pad 2: /ENCA -> /ENCN
- J2 pad 4: /ENCN -> /ENCA
- J7 pad 2: /ENCA -> /ENCN
- J7 pad 4: /ENCN -> /ENCA
- R1 pad 1: /ENCN -> /ENCA
- R3 pad 1: /ENCA -> /ENCN
Routing:
- net +3.3V: track 134.1 -> 169.8 mm, vias 4 -> 0
- net /DRV_EN#: track 53.5 -> 55.4 mm
- net /ENCB: track 34.5 -> 36.4 mm
- net /ENCN: track 36.2 -> 37.9 mm
- net /OV: track 83.6 -> 82.7 mm
- net GND: vias 51 -> 50
- added copper zone on F.Cu, net /OV_D

Commit message: pretty much done with layout, review time
Parts:
- removed J6: Conn_01x06, Connector_JST:JST_XH_B6B-XH-A_1x06_P2.50mm_Vertical
- removed J7: Conn_01x05, Connector_JST:JST_XH_B5B-XH-A_1x05_P2.50mm_Vertical
- added QR*****: tmc2240-breakout, https://github.com/Gherkin/tmc2240-breakout, B.Cu at (159.0, 99.0)
- added R28: 24k, Resistor_SMD:R_0201_0603Metric, F.Cu at (133.0, 98.5)
- added R29: 24k, Resistor_SMD:R_0201_0603Metric, F.Cu at (133.0, 99.8)
- added REF**: qr, qr:qr, F.Cu at (104.0, 90.0)
- added TP22: TestPoint_Alt, TestPoint:TestPoint_THTPad_1.0x1.0mm_Drill0.5mm, F.Cu at (137.0, 99.0)
Routing:
- net /OV: track 82.7 -> 88.2 mm, vias 4 -> 5
- net /DIAG1#: track 68.4 -> 72.6 mm, vias 6 -> 7
- net /DIAG0#: track 63.4 -> 66.6 mm
- net +3.3V: track 169.8 -> 172.5 mm
Other:
- outline, holes or cut-outs redrawn
- board text added: "%%DATE%%"
- board text added: "4.5-36V"
- board text added: "52 mm (c-c)"
- board text added: "M3"
- board text added: "TMC2240 BREAKOUT"
- board text added: "Ver: %%GITHASH%%"
