File: tmc2240-breakout.kicad_sch (KiCad schematic)
At the start: 92 parts, among them J1 Conn_01x06, J2 Conn_01x05, J3 Conn_01x02, J4 Conn_01x02, J5 Conn_01x17, J6 Conn_01x06, J7 Conn_01x05, J8 Conn_01x02, Q10 2N7002, Q11 2N7002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

Commit message: pretty much done with layout, review time
Parts:
- added R28, R29: 24k, Resistor_SMD:R_0201_0603Metric, symbol Device:R
- added TP22: TestPoint_Alt, TestPoint:TestPoint_THTPad_1.0x1.0mm_Drill0.5mm, symbol Connector:TestPoint_Alt
Connections:
- net +3.3V: now also R28.1, R29.1
- net DIAG0#: now also R28.2
- net DIAG1#: now also R29.2
- net GND: now also TP22.1
Other:
- note added: "Design Note: DIAG0/1 used as default OD"
- note added: "Design Note: IREF as TMC2240-eval"
